File: alys-keyboard.kicad_sch (KiCad schematic)
At the start: 44 parts, among them SW10 SW_Push, SW10_r1 SW_Push, SW11 SW_Push, SW11_r1 SW_Push, SW12 SW_Push, SW12_r1 SW_Push, SW13_r1 SW_Push, SW14 SW_Push, SW14_r1 SW_Push, SW15 SW_Push, SW15_r1 SW_Push, SW16 SW_Push, SW16_r1 SW_Push, SW17 SW_Push, SW17_r1 SW_Push, SW18 SW_Push, SW18_r1 SW_Push, SW2 SW_Push, SW20 SW_Push, SW21 SW_Push, SW2_r1 SW_Push, SW3 SW_Push, SW3_r1 SW_Push, SW4 SW_Push, SW4_r1 SW_Push, SW5 SW_Push, SW5_r1 SW_Push, SW6 SW_Push, SW6_r1 SW_Push, SW7_r1 SW_Push, SW8 SW_Push, SW8_r1 SW_Push, SW9 SW_Push, SW9_r1 SW_Push, U1 ProMicro-kbd, U2 ProMicro-kbd

Commit message: schematic design
added 6x6 keyboard matrix
Parts:
- removed SW10_r1, SW11_r1, SW12_r1, SW13_r1, SW14_r1, SW15_r1, SW16_r1, SW17_r1, SW18_r1, SW2_r1, SW3_r1, SW4_r1, SW5_r1, SW6_r1, SW7_r1, SW8_r1, SW9_r1: SW_Push, Kailh:SW_PG1350_rev_DPB, symbol Switch:SW_Push
- added D1, D10, D11, D12, D13, D14, D15, D16, D17, D18, D19, D2, D20, D21, D22, D23, D24, D25, D26, D27, D28, D29, D3, D30, D31, D32, D33, D34, D35, D36, D37, D38, D39, D4, D40, D41, D42, D43, D44, D45, D46, D47, D48, D49, D5, D50, D51, D52, D53, D54, D55, D56, D57, D58, D59, D6, D60, D61, D62, D63, D64, D65, D66, D67, D68, D69, D7, D70, D71, D72, D8, D9: 1N4148W, Diode_SMD:D_SOD-123, symbol Diode:1N4148W
- added SW13, SW19, SW22, SW23, SW24, SW25, SW26, SW27, SW28, SW29, SW30, SW31, SW32, SW33, SW34, SW35, SW36, SW37, SW38, SW39, SW40, SW41, SW42, SW43, SW44, SW45, SW46, SW47, SW48, SW49, SW50, SW51, SW52, SW53, SW54, SW55, SW56, SW57, SW58, SW59, SW60, SW61, SW62, SW63, SW64, SW65, SW66, SW67, SW68, SW69, SW7, SW70, SW71, SW72, SW73: SW_Push, Kailh:SW_PG1350_rev_DPB, symbol Switch:SW_Push
Connections:
- net gnd: no longer BatGND4.1, RSW2.1, SW10.2, SW11.2, SW12.2, SW14.2, SW15.2, SW16.2, SW17.2, SW18.2, SW2.2, SW20.2, SW21.2, SW3.2, SW4.2, SW5.2, SW6.2, SW8.2, SW9.2, U2.23 (GND), U2.3 (GND), U2.4 (GND)
- net raw: no longer SW_POWERR1.3 (C), U2.24 (RAW)
- net Switch1 renamed COL0
- net COL0: now also SW14.1, SW20.1, SW8.1, U1.13 (B6), SW26.1, SW32.1; no longer U1.9 (D7)
- net Switch10: no longer names the net of U1.1 (TX)
- net Switch10: no longer SW12.1
- net Switch10_r: no longer names the net of U2.1 (TX)
- net Switch11: no longer names the net of U1.5 (SDA)
- net Switch11: no longer SW14.1
- net Switch11_r: no longer names the net of U2.5 (SDA)
- net Switch12: no longer names the net of U1.6 (SCL)
- net Switch12: no longer SW15.1
- net Switch12_r: no longer names the net of U2.6 (SCL)
- net Switch13 renamed COL2
- net COL2: now also SW10.1, SW4.1, U1.15 (B3), SW22.1, SW28.1, SW34.1; no longer U1.7 (D4)
- net Switch13_r renamed ROW0_r
- net ROW0_r: now also D37.1 (K), D43.1 (K), D49.1 (K), D55.1 (K), D61.1 (K), D67.1 (K)
- net Switch14 renamed COL3
- net COL3: now also SW11.1, SW5.1, U1.16 (B1), SW23.1, SW29.1, SW35.1; no longer U1.8 (C6)
- net Switch14_r renamed ROW1_r
- net ROW1_r: now also D38.1 (K), D44.1 (K), D50.1 (K), D56.1 (K), D62.1 (K), D68.1 (K)
- net Switch15 renamed COL4
- net COL4: now also SW12.1, SW6.1, U1.17 (F7), SW24.1, SW30.1, SW36.1; no longer U1.10 (E6)
- net Switch15_r renamed ROW3_r
- net ROW3_r: now also D40.1 (K), D46.1 (K), D52.1 (K), D58.1 (K), D64.1 (K), D70.1 (K)
- net Switch16 renamed ROW4
- net ROW4: now also D25.1 (K), D26.1 (K), D27.1 (K), D28.1 (K), D29.1 (K), D30.1 (K); no longer SW20.1
- net Switch16_r renamed ROW4_r
- net ROW4_r: now also D41.1 (K), D47.1 (K), D53.1 (K), D59.1 (K), D65.1 (K), D71.1 (K)
- net Switch17 renamed COL1
- net COL1: now also SW15.1, SW3.1, SW9.1, U1.14 (B2), SW27.1, SW33.1; no longer U1.12 (B5)
- net Switch17_r renamed ROW5_r
- net ROW5_r: now also D42.1 (K), D48.1 (K), D54.1 (K), D60.1 (K), D66.1 (K), D72.1 (K)
- net Switch18: no longer names the net of U1.2 (RX)
- net Switch18_r: no longer names the net of U2.2 (RX)
- net Switch1_r renamed ROW2_r
- net ROW2_r: now also D39.1 (K), D45.1 (K), D51.1 (K), D57.1 (K), D63.1 (K), D69.1 (K)
- removed net Switch2: SW3.1, U1.17 (F7)
- net Switch2_r renamed COL4_r
- net COL4_r: now also SW62.1, SW63.1, SW64.1, SW65.1, SW66.1, SW67.1
- net Switch3 renamed COL5
- net COL5: now also SW13.1, SW19.1, SW25.1, SW31.1, SW37.1, SW7.1; no longer SW4.1
- net Switch3_r renamed COL5_r
- net COL5_r: now also SW68.1, SW69.1, SW70.1, SW71.1, SW72.1, SW73.1
- net Switch4: no longer names the net of U1.19 (F5)
- net Switch4: no longer SW5.1
- net Switch4_r: no longer names the net of U2.19 (F5)
- net Switch5: no longer names the net of U1.20 (F4)
- net Switch5: no longer SW6.1
- net Switch5_r: no longer names the net of U2.20 (F4)
- removed net Switch6: SW8.1, U1.16 (B1)
- net Switch6_r renamed COL3_r
- net COL3_r: now also SW56.1, SW57.1, SW58.1, SW59.1, SW60.1, SW61.1
- removed net Switch7: SW9.1, U1.15 (B3)
- net Switch7_r renamed COL2_r
- net COL2_r: now also SW50.1, SW51.1, SW52.1, SW53.1, SW54.1, SW55.1
- removed net Switch8: SW10.1, U1.14 (B2)
- net Switch8_r renamed COL1_r
- net COL1_r: now also SW44.1, SW45.1, SW46.1, SW47.1, SW48.1, SW49.1
- removed net Switch9: SW11.1, U1.13 (B6)
- net Switch9_r renamed COL0_r
- net COL0_r: now also SW38.1, SW39.1, SW40.1, SW41.1, SW42.1, SW43.1
- new net: D1.2 (A), SW2.2
- new net: D43.2 (A), SW44.2
- new net: D19.2 (A), SW20.2
- new net: D68.2 (A), SW69.2
- new net: D21.2 (A), SW22.2
- new net: D15.2 (A), SW16.2
- new net: D55.2 (A), SW56.2
- new net: D40.2 (A), SW41.2
- new net: D70.2 (A), SW71.2
- new net: D18.2 (A), SW19.2
- new net: D24.2 (A), SW25.2
- new net: D29.2 (A), SW30.2
- new net: D41.2 (A), SW42.2
- new net: D72.2 (A), SW73.2
- new net: D14.2 (A), SW15.2
- new net: D9.2 (A), SW10.2
- new net: D39.2 (A), SW40.2
- new net: D64.2 (A), SW65.2
- new net: D50.2 (A), SW51.2
- new net: D25.2 (A), SW26.2
- new net: D23.2 (A), SW24.2
- new net: D26.2 (A), SW27.2
- new net: D62.2 (A), SW63.2
- new net: D3.2 (A), SW4.2
- new net: D58.2 (A), SW59.2
- new net: D66.2 (A), SW67.2
- new net: D44.2 (A), SW45.2
- new net: D8.2 (A), SW9.2
- new net: D42.2 (A), SW43.2
- new net: D38.2 (A), SW39.2
- new net: D56.2 (A), SW57.2
- new net: D35.2 (A), SW36.2
- new net: D46.2 (A), SW47.2
- new net: D48.2 (A), SW49.2
- new net: D31.2 (A), SW32.2
- new net: D51.2 (A), SW52.2
- new net: D30.2 (A), SW31.2
- new net: D5.2 (A), SW6.2
- new net: D12.2 (A), SW13.2
- new net: D36.2 (A), SW37.2
- new net: D6.2 (A), SW7.2
- new net: D32.2 (A), SW33.2
- new net: D37.2 (A), SW38.2
- new net: D67.2 (A), SW68.2
- new net: D20.2 (A), SW21.2
- new net: D11.2 (A), SW12.2
- new net: D61.2 (A), SW62.2
- new net: D47.2 (A), SW48.2
- new net: D4.2 (A), SW5.2
- new net: D33.2 (A), SW34.2
- new net: D22.2 (A), SW23.2
- new net: D34.2 (A), SW35.2
- new net: D28.2 (A), SW29.2
- new net: D49.2 (A), SW50.2
- new net: D16.2 (A), SW17.2
- new net: D52.2 (A), SW53.2
- new net: D17.2 (A), SW18.2
- new net: D65.2 (A), SW66.2
- new net: D71.2 (A), SW72.2
- new net: D7.2 (A), SW8.2
- new net: D69.2 (A), SW70.2
- new net: D2.2 (A), SW3.2
- new net: D13.2 (A), SW14.2
- new net: D27.2 (A), SW28.2
- new net: D63.2 (A), SW64.2
- new net: D57.2 (A), SW58.2
- new net: D59.2 (A), SW60.2
- new net: D45.2 (A), SW46.2
- new net: D10.2 (A), SW11.2
- new net: D60.2 (A), SW61.2
- new net: D53.2 (A), SW54.2
- new net: D54.2 (A), SW55.2
- new net ROW0: D1.1 (K), D2.1 (K), D3.1 (K), D4.1 (K), D5.1 (K), D6.1 (K), U1.7 (D4)
- new net ROW1: D10.1 (K), D11.1 (K), D12.1 (K), D7.1 (K), D8.1 (K), D9.1 (K), U1.8 (C6)
- new net ROW2: D13.1 (K), D14.1 (K), D15.1 (K), D16.1 (K), D17.1 (K), D18.1 (K), U1.9 (D7)
- new net ROW3: D19.1 (K), D20.1 (K), D21.1 (K), D22.1 (K), D23.1 (K), D24.1 (K), U1.10 (E6)
- new net ROW5: D31.1 (K), D32.1 (K), D33.1 (K), D34.1 (K), D35.1 (K), D36.1 (K), U1.12 (B5)
- new net gnd_r: BatGND4.1, RSW2.1, U2.23 (GND), U2.3 (GND), U2.4 (GND)
- new net raw_r: SW_POWERR1.3 (C), U2.24 (RAW)
Other:
- moved on the sheet: Bat+r1, BatGND4, RSW2, SW2, SW_POWERR1, U2
